File: Hardware/PCBs/actuation_board_v2/Servos.kicad_sch (KiCad schematic)
At the start: 4 parts

Commit message: Final schematic
Parts:
- J1: renamed from J?; value SERVO -> SERVO1
- J2: renamed from J?; value SERVO -> SERVO2
- J3: renamed from J?; value SERVO -> SERVO3
- J4: renamed from J?; value SERVO -> SERVO4
Connections:
- net +7.4V: now also J1.2 (Pin_2), J2.2 (Pin_2), J3.2 (Pin_2), J4.2 (Pin_2); no longer J1.3 (Pin_3), J2.3 (Pin_3), J3.3 (Pin_3), J4.3 (Pin_3)
- net GND: now also J1.3 (Pin_3), J2.3 (Pin_3), J3.3 (Pin_3), J4.3 (Pin_3); no longer J1.1 (Pin_1), J2.1 (Pin_1), J3.1 (Pin_1), J4.1 (Pin_1)
- net S1: now also J1.1 (Pin_1); no longer J1.2 (Pin_2)
- net S2: now also J2.1 (Pin_1); no longer J2.2 (Pin_2)
- net S3: now also J3.1 (Pin_1); no longer J3.2 (Pin_2)
- net S4: now also J4.1 (Pin_1); no longer J4.2 (Pin_2)

Commit message: Finished schematic and PCB
Parts:
- added C4: 100nF, Capacitor_SMD:C_0603_1608Metric_Pad1.08x0.95mm_HandSolder, symbol Device:C
- added C5: 470uF, Capacitor_SMD:CP_Elec_8x10.5, symbol Device:C_Polarized
- J1, J2, J3, J4: footprint Connector_Molex:Molex_Nano-Fit_105309-xx03_1x03_P2.50mm_Vertical -> Connector_PinHeader_2.54mm:PinHeader_1x03_P2.54mm_Vertical
Connections:
- net +7.4V: now also C5.1
- net GND: now also C4.2
- new net: C4.1, C5.2
