File: Hardware/PCBs/actuation_board_v2/actuation_board2.kicad_sch (KiCad schematic)
At the start: 2 parts, among them J6 Conn_01x11_Socket, U2 ESP32-S3-DevKitC

Commit message: Final schematic
Connections:
- no-connect marks 0 -> 22

Commit message: Finished schematic and PCB
Parts:
- added C2, C3: 10uF, Capacitor_SMD:C_0603_1608Metric_Pad1.08x0.95mm_HandSolder, symbol Device:C_Polarized
- added F1: 15A, Fuse:Fuse_1206_3216Metric_Pad1.42x1.75mm_HandSolder, symbol Device:Fuse
- added J7: Conn_01x02_Pin, Connector_AMASS:AMASS_XT60PW-M_1x02_P7.20mm_Horizontal, symbol Connector:Conn_01x02_Pin
- added U3: R-78E5.0-1.0, Converter_DCDC:Converter_DCDC_RECOM_R-78E-0.5_THT, symbol Regulator_Switching:R-78E5.0-1.0
- J6: footprint (none) -> Connector_PinSocket_2.54mm:PinSocket_1x11_P2.54mm_Vertical
Connections:
- net +5V: now also C3.1, U3.3 (OUT)
- net GND: now also C2.2, C3.2, J7.2 (Pin_2), U3.2 (GND)
- new net: F1.2, J7.1 (Pin_1)
- new net +7.4V: C2.1, F1.1, U3.1 (IN)
Other:
- moved on the sheet: J6, U2
